File: Lab Controller Board/Lab Controller Board v04.brd (EAGLE design)
At the start: 50 x 50 mm, 52 parts, among them Q2 MMBT5088, Q3 100A/100V, Q4 MMBT5088, Q5 100A/100V, Q6 MMBT5088, Q7 100A/100V, Q8 MMBT5088, U1 ATMEGA328P_TQFP, U2 CH340G, Y1 16MHZ

Commit message: Working on Lab LED
Parts:
- moved R4 83.9 mm to (91.8, 19.7)
- moved STANDOFF1 73.3 mm to (77.5, 35.2)
- moved JP8 72.0 mm to (77.0, 16.0), turned to 90 degrees
- moved Q2 68.0 mm to (92.3, 29.5)
- moved R3 67.2 mm to (70.2, 53.2), turned to 270 degrees
- moved Q4 67.1 mm to (81.4, 29.8)
- moved R2 66.6 mm to (85.0, 22.4)
- moved R9 64.3 mm to (73.0, 19.0), turned to 180 degrees
- moved R10 64.0 mm to (73.0, 15.8), turned to 180 degrees
- moved JP7 63.7 mm to (66.3, 34.2), turned to 270 degrees
- moved R1 62.9 mm to (67.4, 53.1), turned to 270 degrees
- moved MC7805CD2TR4 62.2 mm to (66.0, 52.3), turned to 90 degrees
- moved Q8 61.1 mm to (94.8, 35.9)
- moved R7 59.4 mm to (64.8, 53.1), turned to 270 degrees
- moved R8 58.3 mm to (87.0, 37.2)
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Connections:
- new net N$12: JP7.1, JP7.10, JP7.11, JP7.12, JP7.2, JP7.3, JP7.4, JP7.5, JP7.6, JP7.7, JP7.8, JP7.9
- new net N$15: U1.1, U1.10, U1.11, U1.12, U1.13, U1.14, U1.15, U1.16, U1.19, U1.2, U1.22, U1.23, U1.24, U1.25, U1.26, U1.27, U1.28, U1.30, U1.31, U1.32, U1.9
- new net POWER_LED: LED1.2, R15.1
- net N$10: no longer LED1.2
Routing:
- net 12V: track 120.1 -> 0.00 mm
- net PWM_B1: track 69.7 -> 0.00 mm
- net PWM_B: track 54.9 -> 0.00 mm
- net PWM_B3: track 54.0 -> 0.00 mm
- net PWM_B2: track 48.8 -> 0.00 mm
- net FET_SOURCE1: track 35.9 -> 0.00 mm
- net N$5: track 29.2 -> 0.00 mm, vias 1 -> 0
- net FET_SOURCE2: track 28.4 -> 0.00 mm
- net FET_SOURCE: track 27.4 -> 0.00 mm
- net FET_SOURCE3: track 26.9 -> 0.00 mm
- net N$7: track 21.9 -> 0.00 mm, vias 1 -> 0
- net LED_DRAIN2: track 18.1 -> 0.00 mm
- net N$10: track 15.5 -> 0.00 mm, vias 1 -> 0
- net SDA: track 13.7 -> 0.00 mm
- net LED_DRAIN3: track 12.3 -> 0.00 mm
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