File: Lab Controller Board/Lab Controller Board v05.sch (EAGLE design)
At the start: 51 parts, among them Q2 NPN - 2N5088, Q3 MOSFET-NCHANNELFQP30N06L, Q4 NPN - 2N5088, Q5 MOSFET-NCHANNELFQP30N06L, Q6 NPN - 2N5088, Q7 MOSFET-NCHANNELFQP30N06L, Q8 NPN - 2N5088, U1 ATMEGA328P_TQFP, U2 CH340G, Y1 16MHZ

Commit message: Working on Lab LED
Parts:
- removed JP6, JP7: (no value), SparkFun-Connectors:M12PTH
- removed R15: 330, resistor:R-US_R0402
- FQP30N06L, Q3, Q5, Q7: value MOSFET-NCHANNELFQP30N06L -> 100A/100V; device SparkFun-DiscreteSemi:MOSFET-NCHANNELFQP30N06L -> SparkFun-DiscreteSemi:MOSFET-NCHANNELPSMN7R0
- Q2, Q4, Q6, Q8: value NPN - 2N5088 -> MMBT5088; device SparkFun-DiscreteSemi:TRANSISTOR_NPNTO92 -> SparkFun-DiscreteSemi:TRANSISTOR_NPNMMBT5088
Connections:
- removed net N$10: JP6.3, LED1.RED-A
- removed net N$14: R15.2, U1.PB5(SCK)
- removed net N$3: JP6.10
- removed net N$30: U2.CTS, U2.DCD, U2.DSR, U2.RI, U2.RS232, U2.RTS
- removed net N$4: JP6.9
- removed net RX: JP6.11
- removed net TX: JP6.12
- new net 0: U1.PD0(RXD)
- new net 1: U1.PD1(TXD)
- new net 10: U1.PB2(SS/OC1B)
- new net 11: U1.PB3(MOSI/OC2)
- new net 12: U1.PB4(MISO)
- new net 13: LED1.RED-A, U1.PB5(SCK)
- new net 2: U1.PD2(INT0)
- new net 3: U1.PD3(INT1)
- new net 4: U1.PD4(XCK/T0)
- new net 5: U1.PD5(T1)
- new net 6: U1.PD6(AIN0)
- new net 7: U1.PD7(AIN1)
- new net 8: U1.PB0(ICP)
- new net A0: U1.PC0(ADC0)
- new net A1: U1.PC1(ADC1)
- new net A2: U1.PC2(ADC2)
- new net A3: U1.PC3(ADC3)
- new net A4: U1.PC4(ADC4/SDA)
- new net A5: U1.PC5(ADC5/SCL)
- new net A6: U1.ADC6
- new net A7: U1.ADC7
- new net X0: C7.1, Q1.2, U2.XO
- new net X1: C6.1, Q1.1, U2.XI
- net 9: now also U1.PB1(OC1A); no longer JP6.2
- net APM_PIN_3: no longer JP6.7
- net APM_PIN_5: no longer JP6.5
- net APM_PIN_6: no longer JP6.4
- net APM_PIN_9: no longer JP6.1
- net N$32: no longer C6.1, C7.1, Q1.1, Q1.2, U2.XI, U2.XO
- net N$5: no longer JP6.8
- net N$7: no longer JP6.6
Other:
- moved on the sheet: C5, JP8, LED1, R10, R11, R12, R13, R14, R9, S1

Commit message: Working
Connections:
- removed net 5V: J1.VCC, R10.2, R9.2, U2.VCC
- net VCC: now also J1.VCC, R10.2, R9.2, U2.VCC
Changed lines of the file:
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@@
-</segment>
-</net>
-<net name="5V" class="0">
-<segment>
-<wire x1="66.04" y1="45.72" x2="55.88" y2="45.72" width="0.1524" layer="91"/>
-<pinref part="J1" gate="G$1" pin="VCC"/>
-<label x="58.42" y="45.72" size="1.778" layer="95"/>
-</segment>
-<segment>
-<pinref part="U2" gate="G$1" pin="VCC"/>
-<wire x1="91.44" y1="76.2" x2="99.06" y2="76.2" width="0.1524" layer="91"/>
-<label x="96.52" y="76.2" size="1.778" layer="95"/>
-</segment>
-<segment>
-<pinref part="R9" gate="G$1" pin="2"/>
-<wire x1="149.86" y1="132.08" x2="160.02" y2="132.08" width="0.1524" layer="91"/>
-<wire x1="160.02" y1="132.08" x2="160.02" y2="127" width="0.1524" layer="91"/>
-<pinref part="R10" gate="G$1" pin="2"/>
-<wire x1="157.48" y1="127" x2="160.02" y2="127" width="0.1524" layer="91"/>
-<label x="162.56" y="139.7" size="1.778" layer="95" rot="R180"/>
-<wire x1="160.02" y1="132.08" x2="160.02" y2="137.16" width="0.1524" layer="91"/>
 </segment>
 </net>
@@
 <wire x1="185.42" y1="71.12" x2="182.88" y2="71.12" width="0.1524" layer="91"/>
 </segment>
+<segment>
+<pinref part="R9" gate="G$1" pin="2"/>
+<wire x1="149.86" y1="132.08" x2="160.02" y2="132.08" width="0.1524" layer="91"/>
+<wire x1="160.02" y1="132.08" x2="160.02" y2="127" width="0.1524" layer="91"/>
+<pinref part="R10" gate="G$1" pin="2"/>
+<wire x1="157.48" y1="127" x2="160.02" y2="127" width="0.1524" layer="91"/>
+<label x="162.56" y="139.7" size="1.778" layer="95" rot="R180"/>
+<wire x1="160.02" y1="132.08" x2="160.02" y2="137.16" width="0.1524" layer="91"/>
+</segment>
+<segment>
+<pinref part="U2" gate="G$1" pin="VCC"/>
+<wire x1="91.44" y1="76.2" x2="99.06" y2="76.2" width="0.1524" layer="91"/>
+<label x="96.52" y="76.2" size="1.778" layer="95"/>
+</segment>
+<segment>
+<wire x1="66.04" y1="45.72" x2="55.88" y2="45.72" width="0.1524" layer="91"/>
+<pinref part="J1" gate="G$1" pin="VCC"/>
+<label x="58.42" y="45.72" size="1.778" layer="95"/>
+</segment>
 </net>

Commit message: Lab Controller
Parts:
- removed J1: (no value), SparkFun-Connectors:USB_MICROB_PLUGCONN-11752
- removed R16, R17: 1k, resistor:R-US_R0402
- added C8: 0.1uF, resistor:C-USC0402
- added CN1: (no value), adafruit:USBMINIB
Connections:
- removed net 0: U1.PD0(RXD)
- removed net 1: U1.PD1(TXD)
- removed net APM_PIN_3: R3.1
- removed net APM_PIN_5: R1.1
- removed net APM_PIN_6: R7.1
- removed net APM_PIN_9: R5.1
- removed net N$5: LED1.BLU-A
- removed net N$7: LED1.GRN-A
- new net ID: CN1.ID
- net 10: now also R1.1
- net 11: now also R3.1
- net 5: now also R5.1
- net 9: now also R7.1
- net A1: now also LED1.GRN-A
- net A2: now also LED1.BLU-A
- net D+: now also CN1.D+; no longer J1.D+
- net D-: now also CN1.D-; no longer J1.D-
- net GND: now also C8.2, CN1.GND; no longer J1.GND, J1.ID, J1.SHIELD
- net U2_RX: now also U1.PD1(TXD); no longer R17.2
- net U2_TX: now also U1.PD0(RXD); no longer R16.2
- net VCC: now also C8.1, CN1.VBUS; no longer J1.VCC
Other:
- moved on the sheet: C3

Commit message: Lab controller
Changed lines of the file:
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@@
 <grid distance="0.1" unitdist="inch" unit="inch" style="lines" multiple="1" display="no" altdistance="0.01" altunitdist="inch" altunit="inch"/>
 <layers>
-<layer number="1" name="Top" color="4" fill="1" visible="yes" active="no"/>
-<layer number="16" name="Bottom" color="1" fill="1" visible="yes" active="no"/>
-<layer number="17" name="Pads" color="2" fill="1" visible="yes" active="no"/>
-<layer number="18" name="Vias" color="2" fill="1" visible="yes" active="no"/>
-<layer number="19" name="Unrouted" color="6" fill="1" visible="yes" active="no"/>
-<layer number="20" name="Dimension" color="15" fill="1" visible="yes" active="no"/>
-<layer number="21" name="tPlace" color="7" fill="1" visible="yes" active="no"/>
-<layer number="22" name="bPlace" color="7" fill="1" visible="yes" active="no"/>
-<layer number="23" name="tOrigins" color="15" fill="1" visible="yes" active="no"/>
-<layer number="24" name="bOrigins" color="15" fill="1" visible="yes" active="no"/>
-<layer number="25" name="tNames" color="7" fill="1" visible="yes" active="no"/>
-<layer number="26" name="bNames" color="7" fill="1" visible="yes" active="no"/>
-<layer number="27" name="tValues" color="7" fill="1" visible="yes" active="no"/>
-<layer number="28" name="bValues" color="7" fill="1" visible="yes" active="no"/>
+<layer number="1" name="Top" color="4" fill="1" visible="no" active="no"/>
+<layer number="16" name="Bottom" color="1" fill="1" visible="no" active="no"/>
+<layer number="17" name="Pads" color="2" fill="1" visible="no" active="no"/>
+<layer number="18" name="Vias" color="2" fill="1" visible="no" active="no"/>
+<layer number="19" name="Unrouted" color="6" fill="1" visible="no" active="no"/>
+<layer number="20" name="Dimension" color="15" fill="1" visible="no" active="no"/>
+<layer number="21" name="tPlace" color="7" fill="1" visible="no" active="no"/>
+<layer number="22" name="bPlace" color="7" fill="1" visible="no" active="no"/>
+<layer number="23" name="tOrigins" color="15" fill="1" visible="no" active="no"/>
+<layer number="24" name="bOrigins" color="15" fill="1" visible="no" active="no"/>
+<layer number="25" name="tNames" color="7" fill="1" visible="no" active="no"/>
+<layer number="26" name="bNames" color="7" fill="1" visible="no" active="no"/>
+<layer number="27" name="tValues" color="7" fill="1" visible="no" active="no"/>
+<layer number="28" name="bValues" color="7" fill="1" visible="no" active="no"/>
 <layer number="29" name="tStop" color="7" fill="3" visible="no" active="no"/>
 <layer number="30" name="bStop" color="7" fill="6" visible="no" active="no"/>
@@
 <layer number="35" name="tGlue" color="7" fill="4" visible="no" active="no"/>
 <layer number="36" name="bGlue" color="7" fill="5" visible="no" active="no"/>
-<layer number="37" name="tTest" color="7" fill="1" visible="yes" active="no"/>
-<layer number="38" name="bTest" color="7" fill="1" visible="yes" active="no"/>
+<layer number="37" name="tTest" color="7" fill="1" visible="no" active="no"/>
+<layer number="38" name="bTest" color="7" fill="1" visible="no" active="no"/>
 <layer number="39" name="tKeepout" color="4" fill="11" visible="no" active="no"/>
 <layer number="40" name="bKeepout" color="1" fill="11" visible="no" active="no"/>
@@
 <layer number="44" name="Drills" color="7" fill="1" visible="no" active="no"/>
 <layer number="45" name="Holes" color="7" fill="1" visible="no" active="no"/>
-<layer number="46" name="Milling" color="3" fill="1" visible="yes" active="no"/>
-<layer number="47" name="Measures" color="7" fill="1" visible="yes" active="no"/>
-<layer number="48" name="Document" color="7" fill="1" visible="yes" active="no"/>
-<layer number="49" name="Reference" color="7" fill="1" visible="yes" active="no"/>
-<layer number="50" name="dxf" color="7" fill="1" visible="yes" active="no"/>
-<layer number="51" name="tDocu" color="7" fill="1" visible="yes" active="no"/>
-<layer number="52" name="bDocu" color="7" fill="1" visible="yes" active="no"/>
-<layer number="53" name="tGND_GNDA" color="7" fill="9" visible="yes" active="no"/>
-<layer number="54" name="bGND_GNDA" color="1" fill="9" visible="yes" active="no"/>
-<layer number="56" name="wert" color="7" fill="1" visible="yes" active="no"/>
-<layer number="57" name="tCAD" color="7" fill="1" visible="yes" active="no"/>
-<layer number="59" name="tCarbon" color="7" fill="1" visible="yes" active="no"/>
-<layer number="60" name="bCarbon" color="7" fill="1" visible="yes" active="no"/>
+<layer number="46" name="Milling" color="3" fill="1" visible="no" active="no"/>
+<layer number="47" name="Measures" color="7" fill="1" visible="no" active="no"/>
+<layer number="48" name="Document" color="7" fill="1" visible="no" active="no"/>
+<layer number="49" name="Reference" color="7" fill="1" visible="no" active="no"/>
+<layer number="50" name="dxf" color="7" fill="1" visible="no" active="no"/>
+<layer number="51" name="tDocu" color="7" fill="1" visible="no" active="no"/>
+<layer number="52" name="bDocu" color="7" fill="1" visible="no" active="no"/>
+<layer number="53" name="tGND_GNDA" color="7" fill="9" visible="no" active="no"/>
+<layer number="54" name="bGND_GNDA" color="1" fill="9" visible="no" active="no"/>
+<layer number="56" name="wert" color="7" fill="1" visible="no" active="no"/>
+<layer number="57" name="tCAD" color="7" fill="1" visible="no" active="no"/>
+<layer number="59" name="tCarbon" color="7" fill="1" visible="no" active="no"/>
+<layer number="60" name="bCarbon" color="7" fill="1" visible="no" active="no"/>
 <layer number="90" name="Modules" color="5" fill="1" visible="yes" active="yes"/>
 <layer number="91" name="Nets" color="2" fill="1" visible="yes" active="yes"/>
@@
 <net name="D-" class="0">
 <segment>
+<wire x1="111.76" y1="22.86" x2="121.92" y2="22.86" width="0.1524" layer="91"/>
+<pinref part="CN1" gate="G$1" pin="D-"/>
+<label x="111.76" y="22.86" size="1.778" layer="95"/>
+<wire x1="121.92" y1="22.86" x2="121.92" y2="48.26" width="0.1524" layer="91"/>
+<wire x1="121.92" y1="48.26" x2="55.88" y2="48.26" width="0.1524" layer="91"/>
 <wire x1="66.04" y1="63.5" x2="55.88" y2="63.5" width="0.1524" layer="91"/>
 <pinref part="U2" gate="G$1" pin="D-"/>
-</segment>
-<segment>
-<wire x1="111.76" y1="22.86" x2="119.38" y2="22.86" width="0.1524" layer="91"/>
-<pinref part="CN1" gate="G$1" pin="D-"/>
-<label x="111.76" y="22.86" size="1.778" layer="95"/>
+<wire x1="55.88" y1="48.26" x2="55.88" y2="63.5" width="0.1524" layer="91"/>
 </segment>
 </net>
 <net name="D+" class="0">
 <segment>
-<wire x1="66.04" y1="66.04" x2="55.88" y2="66.04" width="0.1524" layer="91"/>
+<wire x1="66.04" y1="66.04" x2="53.34" y2="66.04" width="0.1524" layer="91"/>
 <pinref part="U2" gate="G$1" pin="D+"/>
-</segment>
-<segment>
-<wire x1="111.76" y1="25.4" x2="119.38" y2="25.4" width="0.1524" layer="91"/>
+<wire x1="53.34" y1="66.04" x2="53.34" y2="45.72" width="0.1524" layer="91"/>
+<wire x1="53.34" y1="45.72" x2="124.46" y2="45.72" width="0.1524" layer="91"/>
+<wire x1="124.46" y1="45.72" x2="124.46" y2="25.4" width="0.1524" layer="91"/>
+<wire x1="111.76" y1="25.4" x2="124.46" y2="25.4" width="0.1524" layer="91"/>
 <pinref part="CN1" gate="G$1" pin="D+"/>
 <label x="111.76" y="25.4" size="1.778" layer="95"/>
