File: Lab Controller Board/Lab Controller Board v09.sch (EAGLE design)
At the start: 47 parts, among them Q2 MMBT5088, Q3 100A/100V, Q4 MMBT5088, Q5 100A/100V, Q6 MMBT5088, Q7 100A/100V, Q8 MMBT5088, U1 ATMEGA328P_TQFP, U2 CH340G, U3 +12v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

Commit message: Added ESP-07, RX/TX level converter, temp probe connection.  Cleaned silkscreen
Parts:
- removed JP8: (no value), SparkFun-Connectors:M02LOCK
- added C10: 10uF, SparkFun-Capacitors:CAP_POL3528
- added C11: 470uF, resistor:CPOL-USD/7343-31W
- added C9: 0.1uF, resistor:C-USC0805K
- added J1: DS18B20, SparkFun-Connectors:M03LOCK
- added Q9: MOSFET-NCHANNELAO3404A, SparkFun-DiscreteSemi:MOSFET-NCHANNELAO3404A
- added R15, R19, R20, R21, R22: 10k, resistor:R-US_R0805W
- added R16: 3.3k, resistor:R-US_R0805W
- added R17: 220, resistor:R-US_R0805W
- added R18: 370, resistor:R-US_R0805W
- added R23: 20k, resistor:R-US_R0805W
- added RESONATOR: 16mhz, crystal:CRYSTALHC49UP
- added U$1: ESP8266-07, lio:ESP8266-07
- added U4: V_REG_317SMD, SparkFun-PowerIC:V_REG_317SMD
- C4, C5, C6, C7: device resistor:C-USC0402 -> resistor:C-USC0805K
- CN1: value (none) -> USB_CON
- JP1: value (none) -> 12V_INPUT
- JP2: value (none) -> LED_THREE
- JP3: value (none) -> LED_TWO
- JP4: value (none) -> LED_ONE
- JP5: value (none) -> LED_FOUR
- Q1: value (none) -> MOSFET-NCHANNELAO3404A; device crystal:CRYSTALHC49UP -> SparkFun-DiscreteSemi:MOSFET-NCHANNELAO3404A
- R10: value 4.7k -> 3.3k; device resistor:R-US_M0805 -> resistor:R-US_R0805W
- R14: device resistor:R-US_R0402 -> resistor:R-US_R0805W
- R9: value 4.7k -> 10k; device resistor:R-US_M0805 -> resistor:R-US_R0805W
Connections:
- removed net 2: U1.PD2(INT0)
- removed net 3: U1.PD3(INT1)
- removed net 4: U1.PD4(XCK/T0)
- removed net 6: U1.PD6(AIN0)
- removed net 7: U1.PD7(AIN1)
- removed net 8: U1.PB0(ICP)
- removed net A0: U1.PC0(ADC0)
- removed net A4: U1.PC4(ADC4/SDA)
- removed net A5: U1.PC5(ADC5/SCL)
- removed net A6: U1.ADC6
- removed net A7: U1.ADC7
- removed net ID: CN1.ID
- removed net N$32: U2.V3
- removed net SCL: JP8.1, R10.1
- removed net SDA: JP8.2, R9.1
- new net 3.35V: C11.+, C9.1, Q1.G, Q9.G, R10.1, R17.2, R21.2, R22.2, U$1.CH_PD, U$1.VCC, U4.OUT
- new net ESP-RX: Q9.D, R19.1, U1.PD7(AIN1)
- new net ESP-TX: Q1.D, R20.1, U1.PD6(AIN0)
- new net N$12: Q1.S, R22.1, U$1.TXD
- new net N$14: R17.1, R18.2, U4.ADJ
- new net N$15: Q9.S, R21.1, U$1.RXD
- new net N$3: R15.1, U$1.REST
- new net N$4: R10.2, U$1.GPIO2
- new net N$5: R16.2, U$1.GPIO15
- net 12: now also R15.2, R23.2
- net A3: now also J1.2, R9.1
- net GND: now also C10.-, C11.-, C9.2, J1.1, J1.3, R16.1, R18.1, R23.1, U$1.GND
- net VCC: now also C10.+, R19.2, R20.2, U4.IN; no longer R10.2
- net X0: now also RESONATOR.2; no longer Q1.2
- net X1: now also RESONATOR.1; no longer Q1.1
Other:
- moved on the sheet: R10, R9
