File: Robinson/robinson_v01.brd (EAGLE design)
At the start: 100 x 80 mm, 31 parts, among them Q1 DMP1045U, Q2 MMBT2222A, U2 MCP73831

Commit message: Finished Robinson schematic
Parts:
- added J3: (no value), SparkFun-Connectors:1X04
- added R14: 240, resistor:R0805
- added R15: 390, resistor:R0805
- J1: value (none) -> 3.7_LIPO
- J2: value (none) -> 3.3-4.5 Motor
- moved 3.3V 16.9 mm to (16.5, 43.2), turned to 270 degrees
Connections:
- net N$1 renamed RESET
- net N$13 renamed TX
- net N$15 renamed RX
- net N$2 renamed HM_RES
- net N$24 renamed RED
- net N$25 renamed GREEN
- net N$26 renamed BLUE
- net N$4 renamed PIO3
- net N$5 renamed MOTOR
- net N$8 renamed BATT_MONT
- removed net N$3: U$1.14
- new net N$9: 3.3V.1, R14.1, R15.2
- new net PA3: J3.3, U$3.10
- new net PB0: J3.1, U$3.2
- new net PB1: J3.2, U$3.3
- new net PIO2: J3.4, U$1.14
- net GND: now also R15.1
- net VCC: now also R14.2
Changed lines of the file:
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@@
 <attribute name="PROD_ID" value="IC-11285" x="7.62" y="21.59" size="1.778" layer="27" rot="R180" display="off"/>
 </element>
-<element name="3.3V" library="SparkFun-PowerIC" package="SOT223" value="V_REG_317SMD" x="12.7" y="26.67" rot="R90"/>
+<element name="3.3V" library="SparkFun-PowerIC" package="SOT223" value="V_REG_317SMD" x="16.51" y="43.18" rot="R270"/>
 <element name="U2" library="SparkFun-PowerIC" package="SOT23-5" value="MCP73831" x="3.81" y="3.81" rot="R180">
 <attribute name="PROD_ID" value="IC-09995" x="3.81" y="3.81" size="1.778" layer="27" rot="R180" display="off"/>
@@
 <element name="R1" library="resistor" package="R0805" value="" x="8.89" y="15.24" rot="R180"/>
 <element name="C1" library="resistor" package="C0805" value="1uF" x="13.97" y="13.97" rot="R180"/>
-<element name="J1" library="SparkFun-Connectors" package="1X02" value="" x="22.86" y="1.27" rot="R90"/>
+<element name="J1" library="SparkFun-Connectors" package="1X02" value="3.7_LIPO" x="22.86" y="1.27" rot="R90"/>
 <element name="Q1" library="SparkFun-DiscreteSemi" package="SOT23-3" value="DMP1045U" x="19.05" y="17.78" rot="R180">
 <attribute name="PROD_ID" value="TRANS-08285" x="19.05" y="17.78" size="1.778" layer="27" rot="R180" display="off"/>
@@
 </element>
 <element name="R11" library="resistor" package="R0805" value="10K" x="7.62" y="17.78"/>
-<element name="J2" library="SparkFun-Connectors" package="1X02" value="" x="1.27" y="13.97" rot="R90"/>
+<element name="J2" library="SparkFun-Connectors" package="1X02" value="3.3-4.5 Motor" x="1.27" y="13.97" rot="R90"/>
 <element name="Q2" library="SparkFun-DiscreteSemi" package="SOT23-3" value="MMBT2222A" x="3.81" y="11.43">
 <attribute name="PROD_ID" value="TRANS-08049" x="3.81" y="11.43" size="1.778" layer="27" display="off"/>
@@
 <element name="R13" library="resistor" package="R0805" value="10M" x="0" y="-11.43"/>
 <element name="C5" library="resistor" package="C0805" value=".1uF" x="0" y="-17.78"/>
+<element name="R14" library="resistor" package="R0805" value="240" x="0" y="-24.13"/>
+<element name="R15" library="resistor" package="R0805" value="390" x="0" y="-30.48"/>
+<element name="J3" library="SparkFun-Connectors" package="1X04" value="" x="0" y="-38.1">
+<attribute name="PROD_ID" value="CONN-09696" x="0" y="-38.1" size="1.778" layer="27" display="off"/>
+</element>
 </elements>
 <signals>
-<signal name="N$3">
+<signal name="PIO2">
 <contactref element="U$1" pad="14"/>
-</signal>
-<signal name="N$4">
+<contactref element="J3" pad="4"/>
+<wire x1="12.31" y1="5.25" x2="7.62" y2="-38.1" width="0" layer="19" extent="1-1"/>
+</signal>
+<signal name="PIO3">
 <contactref element="U$1" pad="13"/>
 <contactref element="R9" pad="2"/>
@@
 <wire x1="7.81" y1="5.25" x2="8.57" y2="30.48" width="0" layer="19" extent="1-1"/>
 </signal>
-<signal name="N$13">
+<signal name="TX">
 <contactref element="U$1" pad="4"/>
 <contactref element="U$3" pad="12"/>
 <wire x1="8.89" y1="18.79" x2="10.81" y2="19.35" width="0" layer="19" extent="1-1"/>
 </signal>
-<signal name="N$15">
+<signal name="RX">
 <contactref element="U$1" pad="2"/>
 <contactref element="U$3" pad="13"/>
@@
 <contactref element="R12" pad="1"/>
 <contactref element="C5" pad="2"/>
+<contactref element="R15" pad="1"/>
 <wire x1="32.07" y1="53.34" x2="32.07" y2="59.69" width="0" layer="19" extent="1-1"/>
 <wire x1="32.07" y1="46.99" x2="32.07" y2="53.34" width="0" layer="19" extent="1-1"/>
@@
 <wire x1="-0.95" y1="-5.08" x2="3.81" y2="5.1101" width="0" layer="19" extent="1-1"/>
 <wire x1="0.95" y1="-17.78" x2="-0.95" y2="-5.08" width="0" layer="19" extent="1-1"/>
+<wire x1="-0.95" y1="-30.48" x2="0.95" y2="-17.78" width="0" layer="19" extent="1-1"/>
 <wire x1="8.57" y1="43.18" x2="18.73" y2="27.94" width="0" layer="19" extent="1-1"/>
 <wire x1="8.57" y1="49.53" x2="8.57" y2="43.18" width="0" layer="19" extent="1-1"/>
@@
 <contactref element="D1" pad="C"/>
 <contactref element="C1" pad="1"/>
-<wire x1="19.63" y1="22.86" x2="15.7988" y2="28.9814" width="0" layer="19" extent="1-1"/>
+<wire x1="19.63" y1="22.86" x2="13.4112" y2="40.8686" width="0" layer="19" extent="1-1"/>
 <wire x1="18.1" y1="18.78" x2="19.63" y2="22.86" width="0" layer="19" extent="1-1"/>
 <wire x1="14.92" y1="13.97" x2="18.1" y2="18.78" width="0" layer="19" extent="1-1"/>
@@
 <contactref element="U$1" pad="9"/>
 <contactref element="R11" pad="2"/>
-<wire x1="11.43" y1="24.39" x2="15.7988" y2="26.67" width="0" layer="19" extent="1-1"/>
+<contactref element="R14" pad="2"/>
+<wire x1="11.43" y1="24.39" x2="13.4112" y2="43.18" width="0" layer="19" extent="1-1"/>
 <wire x1="8.57" y1="17.78" x2="11.43" y2="24.39" width="0" layer="19" extent="1-1"/>
 <wire x1="4.81" y1="5.25" x2="8.57" y2="17.78" width="0" layer="19" extent="1-1"/>
-</signal>
-<signal name="N$24">
+<wire x1="0.95" y1="-24.13" x2="4.81" y2="5.25" width="0" layer="19" extent="1-1"/>
+</signal>
+<signal name="RED">
 <contactref element="LED1" pad="2"/>
 <contactref element="LED2" pad="2"/>
@@
 <wire x1="3.81" y1="18.79" x2="16.37" y2="16.51" width="0" layer="19" extent="1-1"/>
 </signal>
-<signal name="N$25">
+<signal name="GREEN">
 <contactref element="U$3" pad="6"/>
 <contactref element="LED1" pad="1"/>
@@
 <wire x1="16.37" y1="14.81" x2="5.08" y2="24.39" width="0" layer="19" extent="1-1"/>
 </signal>
-<signal name="N$26">
+<signal name="BLUE">
 <contactref element="U$3" pad="7"/>
 <contactref element="LED1" pad="3"/>
@@
 <wire x1="11.57" y1="18.21" x2="6.67" y2="43.18" width="0" layer="19" extent="1-1"/>
 </signal>
-<signal name="N$1">
+<signal name="RESET">
 <contactref element="R9" pad="1"/>
 <contactref element="U$3" pad="4"/>
@@
 <wire x1="19.304" y1="4.445" x2="6.67" y2="17.78" width="0" layer="19" extent="1-1"/>
 </signal>
-<signal name="N$2">
+<signal name="HM_RES">
 <contactref element="R10" pad="1"/>
 <contactref element="U$3" pad="9"/>
 <wire x1="5.08" y1="18.79" x2="6.67" y2="30.48" width="0" layer="19" extent="1-1"/>
 </signal>
-<signal name="N$5">
+<signal name="MOTOR">
 <contactref element="U$3" pad="5"/>
 <contactref element="Q2" pad="1"/>
@@
 <wire x1="6.03" y1="5.08" x2="3.81" y2="12.53" width="0" layer="19" extent="1-1"/>
 </signal>
-<signal name="N$8">
+<signal name="BATT_MONT">
 <contactref element="U$3" pad="11"/>
 <contactref element="R13" pad="1"/>
 <wire x1="-0.95" y1="-11.43" x2="7.62" y2="18.79" width="0" layer="19" extent="1-1"/>
 </signal>
+<signal name="N$9">
+<contactref element="3.3V" pad="1"/>
+<contactref element="R15" pad="2"/>
+<contactref element="R14" pad="1"/>
+<wire x1="-0.95" y1="-24.13" x2="13.4112" y2="45.4914" width="0" layer="19" extent="1-1"/>
+<wire x1="0.95" y1="-30.48" x2="-0.95" y2="-24.13" width="0" layer="19" extent="1-1"/>
+</signal>
+<signal name="PA3">
+<contactref element="U$3" pad="10"/>
+<contactref element="J3" pad="3"/>
+<wire x1="6.35" y1="18.79" x2="5.08" y2="-38.1" width="0" layer="19" extent="1-1"/>
+</signal>
+<signal name="PB0">
+<contactref element="U$3" pad="2"/>
+<contactref element="J3" pad="1"/>
+<wire x1="10.16" y1="24.39" x2="0" y2="-38.1" width="0" layer="19" extent="1-1"/>
+</signal>
+<signal name="PB1">
+<contactref element="U$3" pad="3"/>
+<contactref element="J3" pad="2"/>
+<wire x1="8.89" y1="24.39" x2="2.54" y2="-38.1" width="0" layer="19" extent="1-1"/>
+</signal>
 </signals>

Commit message: Working
Parts:
- added C6: 4.7uF, resistor:C0805
- moved J3 70.7 mm to (26.0, 27.6), turned to 270 degrees
- moved R15 43.9 mm to (20.6, 8.26), turned to 90 degrees
- moved R6 41.7 mm to (23.2, 17.1)
- moved C5 41.5 mm to (21.9, 17.5), flipped to the bottom, turned to 270 degrees
- moved R5 40.1 mm to (12.7, 25.1)
- moved R14 39.9 mm to (17.5, 11.7), turned to 180 degrees
- moved R4 38.1 mm to (12.4, 21.3)
- moved 3.3V 38.1 mm to (16.2, 5.08), turned to 180 degrees
- moved C3 38.1 mm to (1.91, 18.7), turned to 90 degrees
- moved R13 38.0 mm to (21.0, 20.3), flipped to the bottom, turned to 180 degrees
- moved C2 36.1 mm to (5.08, 11.4)
- moved R12 36.0 mm to (21.9, 23.5), flipped to the bottom, turned to 270 degrees
- moved R7 34.5 mm to (23.2, 18.7)
- moved R8 31.7 mm to (23.2, 15.6)
- moved R3 31.5 mm to (12.4, 23.2), turned to 0 degrees
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Connections:
- net GND: now also C6.2
- net VCC: now also C6.1
Routing:
- net 5V: track 0.00 -> 24.5 mm
- net RX: track 0.00 -> 20.5 mm
- net TX: track 0.00 -> 18.4 mm
- net N$19: track 0.00 -> 18.1 mm, vias 0 -> 2
- net VCC: track 0.00 -> 16.2 mm
- net V_BAT: track 0.00 -> 10.7 mm
- net N$7: track 0.00 -> 6.28 mm
- net N$9: track 0.00 -> 6.02 mm
- net N$20: track 0.00 -> 4.59 mm
- net V_BATT: track 0.00 -> 4.47 mm
- added copper zone on layer 1, net GND
- added copper zone on layer 16, net GND
Other:
- board size 100 x 80 mm -> 27.6 x 29.2 mm
