File: Robinson/robinson_v01.sch (EAGLE design)
At the start: 31 parts, among them Q1 DMP1045U, Q2 MMBT2222A, U2 MCP73831

Commit message: Finished Robinson schematic
Parts:
- added J3: (no value), SparkFun-Connectors:M04PTH
- added R14: 240, resistor:R-US_R0805
- added R15: 390, resistor:R-US_R0805
- J1: value (none) -> 3.7_LIPO
- J2: value (none) -> 3.3-4.5 Motor
Connections:
- net N$1 renamed RESET
- net N$13 renamed TX
- net N$15 renamed RX
- net N$2 renamed HM_RES
- net N$24 renamed RED
- net N$25 renamed GREEN
- net N$26 renamed BLUE
- net N$4 renamed PIO3
- net N$5 renamed MOTOR
- net N$8 renamed BATT_MONT
- removed net N$3: U$1.14-PIO2
- new net N$9: 3.3V.ADJ, R14.1, R15.2
- new net PA3: J3.3, U$3.(PCINT3/T0/ADC3)PA3
- new net PB0: J3.1, U$3.(PCINT8/XTAL1/CLKI)PB0
- new net PB1: J3.2, U$3.(PCINT9/XTAL2)PB1
- new net PIO2: J3.4, U$1.14-PIO2
- net GND: now also R15.1
- net VCC: now also R14.2
Changed lines of the file:
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@@
 <part name="GND3" library="SparkFun-Aesthetics" deviceset="GND" device=""/>
 <part name="C1" library="resistor" deviceset="C-US" device="C0805" value="1uF"/>
-<part name="J1" library="SparkFun-Connectors" deviceset="M02" device="PTH"/>
+<part name="J1" library="SparkFun-Connectors" deviceset="M02" device="PTH" value="3.7_LIPO"/>
 <part name="GND4" library="SparkFun-Aesthetics" deviceset="GND" device=""/>
 <part name="Q1" library="SparkFun-DiscreteSemi" deviceset="MOSFET-PCHANNEL" device="" value="DMP1045U"/>
@@
 <part name="R11" library="resistor" deviceset="R-US_" device="R0805" value="10K"/>
 <part name="SUPPLY3" library="SparkFun-Aesthetics" deviceset="VCC" device=""/>
-<part name="J2" library="SparkFun-Connectors" deviceset="M02" device="PTH"/>
+<part name="J2" library="SparkFun-Connectors" deviceset="M02" device="PTH" value="3.3-4.5 Motor"/>
 <part name="GND13" library="SparkFun-Aesthetics" deviceset="GND" device=""/>
 <part name="SUPPLY4" library="SparkFun-Aesthetics" deviceset="V_BATT" device=""/>
@@
 <part name="C5" library="resistor" deviceset="C-US" device="C0805" value=".1uF"/>
 <part name="GND14" library="SparkFun-Aesthetics" deviceset="GND" device=""/>
+<part name="R14" library="resistor" deviceset="R-US_" device="R0805" value="240"/>
+<part name="R15" library="resistor" deviceset="R-US_" device="R0805" value="390"/>
+<part name="GND15" library="SparkFun-Aesthetics" deviceset="GND" device=""/>
+<part name="J3" library="SparkFun-Connectors" deviceset="M04" device="PTH"/>
 </parts>
 <sheets>
@@
 <instance part="C5" gate="G$1" x="81.28" y="-66.04"/>
 <instance part="GND14" gate="1" x="73.66" y="-78.74"/>
+<instance part="R14" gate="G$1" x="127" y="88.9" rot="R90"/>
+<instance part="R15" gate="G$1" x="114.3" y="78.74" rot="R90"/>
+<instance part="GND15" gate="1" x="114.3" y="71.12"/>
+<instance part="J3" gate="G$1" x="99.06" y="48.26" rot="R180"/>
 </instances>
 <busses>
 </busses>
 <nets>
-<net name="N$3" class="0">
-<segment>
-<wire x1="66.04" y1="48.26" x2="48.26" y2="48.26" width="0.1524" layer="91"/>
+<net name="PIO2" class="0">
+<segment>
+<wire x1="81.28" y1="48.26" x2="48.26" y2="48.26" width="0.1524" layer="91"/>
 <pinref part="U$1" gate="G$1" pin="14-PIO2"/>
-</segment>
-</net>
-<net name="N$4" class="0">
+<wire x1="81.28" y1="48.26" x2="81.28" y2="43.18" width="0.1524" layer="91"/>
+<pinref part="J3" gate="G$1" pin="4"/>
+<label x="88.9" y="43.18" size="1.778" layer="95"/>
+<wire x1="81.28" y1="43.18" x2="93.98" y2="43.18" width="0.1524" layer="91"/>
+<label x="50.8" y="48.26" size="1.778" layer="95"/>
+</segment>
+</net>
+<net name="PIO3" class="0">
 <segment>
 <wire x1="71.12" y1="43.18" x2="48.26" y2="43.18" width="0.1524" layer="91"/>
@@
 <pinref part="R9" gate="G$1" pin="2"/>
 <wire x1="71.12" y1="43.18" x2="71.12" y2="38.1" width="0.1524" layer="91"/>
+<label x="50.8" y="43.18" size="1.778" layer="95"/>
 </segment>
 </net>
@@
 <pinref part="R10" gate="G$1" pin="2"/>
 <wire x1="66.04" y1="33.02" x2="66.04" y2="30.48" width="0.1524" layer="91"/>
-</segment>
-</net>
-<net name="N$13" class="0">
+<label x="50.8" y="33.02" size="1.778" layer="95"/>
+</segment>
+</net>
+<net name="TX" class="0">
 <segment>
 <wire x1="-15.24" y1="43.18" x2="5.08" y2="43.18" width="0.1524" layer="91"/>
@@
 <wire x1="53.34" y1="-55.88" x2="-15.24" y2="-55.88" width="0.1524" layer="91"/>
 <wire x1="-15.24" y1="-55.88" x2="-15.24" y2="43.18" width="0.1524" layer="91"/>
-</segment>
-</net>
-<net name="N$15" class="0">
+<label x="50.8" y="-43.18" size="1.778" layer="95"/>
+<label x="-2.54" y="43.18" size="1.778" layer="95"/>
+</segment>
+</net>
+<net name="RX" class="0">
 <segment>
 <wire x1="-12.7" y1="53.34" x2="5.08" y2="53.34" width="0.1524" layer="91"/>
@@
 <wire x1="48.26" y1="-53.34" x2="-12.7" y2="-53.34" width="0.1524" layer="91"/>
 <wire x1="-12.7" y1="-53.34" x2="-12.7" y2="53.34" width="0.1524" layer="91"/>
+<label x="40.64" y="-53.34" size="1.778" layer="95"/>
+<label x="-2.54" y="53.34" size="1.778" layer="95"/>
 </segment>
 </net>
@@
 <wire x1="58.42" y1="38.1" x2="58.42" y2="20.32" width="0.1524" layer="91"/>
 <pinref part="GND11" gate="1" pin="GND"/>
+<label x="50.8" y="38.1" size="1.778" layer="95"/>
 </segment>
 <segment>
@@
 <wire x1="81.28" y1="-76.2" x2="73.66" y2="-76.2" width="0.1524" layer="91"/>
 <junction x="73.66" y="-76.2"/>
+</segment>
+<segment>
+<pinref part="R15" gate="G$1" pin="1"/>
+<pinref part="GND15" gate="1" pin="GND"/>
 </segment>
 </net>
@@
 <segment>
 <pinref part="3.3V" gate="G$1" pin="OUT"/>
-<wire x1="121.92" y1="96.52" x2="132.08" y2="96.52" width="0.1524" layer="91"/>
+<wire x1="121.92" y1="96.52" x2="127" y2="96.52" width="0.1524" layer="91"/>
 <pinref part="SUPPLY1" gate="G$1" pin="VCC"/>
 <label x="121.92" y="96.52" size="1.778" layer="95"/>
+<pinref part="R14" gate="G$1" pin="2"/>
+<wire x1="127" y1="96.52" x2="132.08" y2="96.52" width="0.1524" layer="91"/>
+<wire x1="127" y1="96.52" x2="127" y2="93.98" width="0.1524" layer="91"/>
+<junction x="127" y="96.52"/>
 </segment>
 <segment>
@@
 <wire x1="50.8" y1="17.78" x2="50.8" y2="22.86" width="0.1524" layer="91"/>
 <junction x="-7.62" y="17.78"/>
+<label x="48.26" y="22.86" size="1.778" layer="95"/>
+<label x="-5.08" y="17.78" size="1.778" layer="95"/>
 </segment>
 <segment>
@@
 </segment>
 </net>
-<net name="N$24" class="0">
+<net name="RED" class="0">
 <segment>
 <pinref part="LED1" gate="D1" pin="RED-A"/>
@@
 <wire x1="48.26" y1="-33.02" x2="91.44" y2="-33.02" width="0.1524" layer="91"/>
 <junction x="91.44" y="-33.02"/>
-</segment>
-</net>
-<net name="N$25" class="0">
+<label x="50.8" y="-33.02" size="1.778" layer="95"/>
+</segment>
+</net>
+<net name="GREEN" class="0">
 <segment>
 <pinref part="U$3" gate="G$1" pin="(PCINT7/ICP/OC0B/ADC7)PA7"/>
@@
 <wire x1="93.98" y1="-35.56" x2="101.6" y2="-35.56" width="0.1524" layer="91"/>
 <junction x="93.98" y="-20.32"/>
-</segment>
-</net>
-<net name="N$26" class="0">
+<label x="50.8" y="-27.94" size="1.778" layer="95"/>
+</segment>
+</net>
+<net name="BLUE" class="0">
 <segment>
 <pinref part="U$3" gate="G$1" pin="(PCINT6/OC1A/SDA/MOSI/ADC6)PA6"/>
@@
 <wire x1="96.52" y1="-38.1" x2="101.6" y2="-38.1" width="0.1524" layer="91"/>
 <junction x="96.52" y="-30.48"/>
+<label x="50.8" y="-30.48" size="1.778" layer="95"/>
 </segment>
 </net>
@@
 </segment>
 </net>
-<net name="N$1" class="0">
+<net name="RESET" class="0">
 <segment>
 <pinref part="R9" gate="G$1" pin="1"/>
@@
 <wire x1="71.12" y1="2.54" x2="78.74" y2="2.54" width="0.1524" layer="91"/>
 <wire x1="78.74" y1="2.54" x2="78.74" y2="5.08" width="0.1524" layer="91"/>
-</segment>
-</net>
-<net name="N$2" class="0">
+<label x="50.8" y="-15.24" size="1.778" layer="95"/>
+</segment>
+</net>
+<net name="HM_RES" class="0">
 <segment>
 <pinref part="R10" gate="G$1" pin="1"/>
@@
 <pinref part="U$3" gate="G$1" pin="(PCINT4/T1/SCL/USCK/ADC4)PA4"/>
 <wire x1="66.04" y1="-35.56" x2="48.26" y2="-35.56" width="0.1524" layer="91"/>
-</segment>
-</net>
-<net name="N$5" class="0">
+<label x="50.8" y="-35.56" size="1.778" layer="95"/>
+</segment>
+</net>
+<net name="MOTOR" class="0">
 <segment>
 <pinref part="U$3" gate="G$1" pin="(PCINT10/INT0/OC0A/CKOUT)PB2"/>
@@
 <pinref part="Q2" gate="G$1" pin="B"/>
 <wire x1="109.22" y1="5.08" x2="86.36" y2="5.08" width="0.1524" layer="91"/>
+<label x="50.8" y="-17.78" size="1.778" layer="95"/>
 </segment>
 </net>
@@
 </segment>
 </net>
-<net name="N$8" class="0">
+<net name="BATT_MONT" class="0">
 <segment>
 <pinref part="U$3" gate="G$1" pin="(PCINT2/AIN1/ADC2)PA2"/>
@@
 <wire x1="48.26" y1="-40.64" x2="63.5" y2="-40.64" width="0.1524" layer="91"/>
 <wire x1="63.5" y1="-40.64" x2="63.5" y2="-43.18" width="0.1524" layer="91"/>
-</segment>
-</net>
+<label x="50.8" y="-40.64" size="1.778" layer="95"/>
+</segment>
+</net>
+<net name="N$9" class="0">
+<segment>
+<pinref part="3.3V" gate="G$1" pin="ADJ"/>
+<wire x1="114.3" y1="88.9" x2="114.3" y2="83.82" width="0.1524" layer="91"/>
+<pinref part="R15" gate="G$1" pin="2"/>
+<pinref part="R14" gate="G$1" pin="1"/>
+<wire x1="127" y1="83.82" x2="114.3" y2="83.82" width="0.1524" layer="91"/>
+<junction x="114.3" y="83.82"/>
+</segment>
+</net>
+<net name="PA3" class="0">
+<segment>
+<pinref part="U$3" gate="G$1" pin="(PCINT3/T0/ADC3)PA3"/>
+<wire x1="48.26" y1="-38.1" x2="63.5" y2="-38.1" width="0.1524" layer="91"/>
+<label x="50.8" y="-38.1" size="1.778" layer="95"/>
+</segment>
+<segment>
+<pinref part="J3" gate="G$1" pin="3"/>
+<wire x1="88.9" y1="45.72" x2="93.98" y2="45.72" width="0.1524" layer="91"/>
+<label x="88.9" y="45.72" size="1.778" layer="95"/>
+</segment>
+</net>
+<net name="PB0" class="0">
+<segment>
+<pinref part="U$3" gate="G$1" pin="(PCINT8/XTAL1/CLKI)PB0"/>
+<wire x1="48.26" y1="-22.86" x2="63.5" y2="-22.86" width="0.1524" layer="91"/>
+<label x="50.8" y="-22.86" size="1.778" layer="95"/>
+</segment>
+<segment>
+<pinref part="J3" gate="G$1" pin="1"/>
+<wire x1="88.9" y1="50.8" x2="93.98" y2="50.8" width="0.1524" layer="91"/>
+<label x="88.9" y="50.8" size="1.778" layer="95"/>
+</segment>
+</net>
+<net name="PB1" class="0">
+<segment>
+<pinref part="U$3" gate="G$1" pin="(PCINT9/XTAL2)PB1"/>
+<wire x1="48.26" y1="-20.32" x2="63.5" y2="-20.32" width="0.1524" layer="91"/>
+<label x="50.8" y="-20.32" size="1.778" layer="95"/>
+</segment>
+<segment>
+<pinref part="J3" gate="G$1" pin="2"/>
+<wire x1="88.9" y1="48.26" x2="93.98" y2="48.26" width="0.1524" layer="91"/>
+<label x="88.9" y="48.26" size="1.778" layer="95"/>
+</segment>
+</net>

Commit message: Working
Parts:
- added C6: 4.7uF, resistor:C-USC0805
Connections:
- net GND: now also C6.2
- net VCC: now also C6.1
Changed lines of the file:
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@@
 <part name="GND15" library="SparkFun-Aesthetics" deviceset="GND" device=""/>
 <part name="J3" library="SparkFun-Connectors" deviceset="M04" device="PTH"/>
+<part name="C6" library="resistor" deviceset="C-US" device="C0805" value="4.7uF"/>
+<part name="GND16" library="SparkFun-Aesthetics" deviceset="GND" device=""/>
 </parts>
 <sheets>
@@
 <instance part="GND15" gate="1" x="114.3" y="71.12"/>
 <instance part="J3" gate="G$1" x="99.06" y="48.26" rot="R180"/>
+<instance part="C6" gate="G$1" x="-5.08" y="-17.78"/>
+<instance part="GND16" gate="1" x="-5.08" y="-25.4"/>
 </instances>
 <busses>
@@
 <pinref part="GND15" gate="1" pin="GND"/>
 </segment>
+<segment>
+<pinref part="C6" gate="G$1" pin="2"/>
+<pinref part="GND16" gate="1" pin="GND"/>
+</segment>
 </net>
 <net name="N$20" class="0">
@@
 <segment>
 <pinref part="U$3" gate="G$1" pin="VCC"/>
-<wire x1="-2.54" y1="-15.24" x2="-7.62" y2="-15.24" width="0.1524" layer="91"/>
+<wire x1="-2.54" y1="-15.24" x2="-5.08" y2="-15.24" width="0.1524" layer="91"/>
 <pinref part="SUPPLY2" gate="G$1" pin="VCC"/>
+<wire x1="-5.08" y1="-15.24" x2="-7.62" y2="-15.24" width="0.1524" layer="91"/>
 <wire x1="-7.62" y1="22.86" x2="-7.62" y2="17.78" width="0.1524" layer="91"/>
 <wire x1="-7.62" y1="17.78" x2="-7.62" y2="-15.24" width="0.1524" layer="91"/>
@@
 <label x="48.26" y="22.86" size="1.778" layer="95"/>
 <label x="-5.08" y="17.78" size="1.778" layer="95"/>
-</segment>
-<segment>
+<pinref part="C6" gate="G$1" pin="1"/>
+<junction x="-5.08" y="-15.24"/>
+</segment>
+<segment>
