File: Robinson/robber_v01.brd (EAGLE design)
At the start: 27.6 x 29.2 mm, 37 parts, among them J1 3.7_LIPO, J2 3.3-4.5 Motor, Q1 DMP1045U, Q2 MMBT2222A, U2 MCP73831

Commit message: ROBBER V01
Parts:
- added U$2: (no value), SparkFun-Aesthetics:OSHW-LOGO-L
- moved R10 1.14 mm to (18.4, 14.6), turned to 180 degrees
- moved S1 0.71 mm to (23.2, 3.81)
Routing:
- net PIO3: track 34.0 -> 31.0 mm
- net PIO2: track 19.8 -> 20.4 mm
