File: BoB Board/BoB Brain v03.sch (EAGLE design)
At the start: 35 parts, among them Q1 MOSFET-NCHANNELAO3404A, Q9 MOSFET-NCHANNELAO3404A, U1 ATMEGA328P_TQFP, U3 +12v, U4 V_REG_317SMD, Y1 16MHZ

Commit message: Working on BoB board
Parts:
- removed JP2, JP3, JP4: (no value), SparkFun-Connectors:M12PTH
- added J1, J2, J4: (no value), SparkFun-Connectors:M18_
Connections:
- net N$28 renamed ADC7
- removed net 10: U1.PB2(SS/OC1B)
- removed net 11: U1.PB3(MOSI/OC2)
- removed net 5: U1.PD5(T1)
- removed net 9: U1.PB1(OC1A)
- removed net N$10: JP4.11
- removed net N$13: U1.PC4(ADC4/SDA)
- removed net N$16: JP4.10
- removed net N$17: JP4.9
- removed net N$18: JP4.8
- removed net N$19: JP4.7
- removed net N$20: JP4.6
- removed net N$21: JP4.5
- removed net N$22: JP4.4
- removed net N$23: JP4.3
- removed net N$24: JP4.2
- removed net N$25: JP4.1
- removed net N$26: U1.PC5(ADC5/SCL)
- removed net N$27: U1.ADC6
- removed net N$29: U1.PD3(INT1)
- removed net N$3: U1.PB4(MISO)
- removed net N$30: U1.PD4(XCK/T0)
- removed net N$31: U1.PD6(AIN0)
- removed net N$32: U1.PD7(AIN1)
- removed net N$33: U1.PB0(ICP)
- removed net N$5: U1.PC3(ADC3)
- removed net N$7: JP4.12
- new net 10~: J2.2, U1.PB2(SS/OC1B)
- new net 11~: J2.1, U1.PB3(MOSI/OC2)
- new net 12: J2.6, U1.PB4(MISO)
- new net 3~: J2.11, U1.PD3(INT1)
- new net 4: J2.10, U1.PD4(XCK/T0)
- new net 5~: J2.9, U1.PD5(T1)
- new net 6~: J2.4, U1.PD6(AIN0)
- new net 7: J2.8, U1.PD7(AIN1)
- new net 8: J2.7, U1.PB0(ICP)
- new net 9~: J2.3, U1.PB1(OC1A)
- new net A3: J2.15, U1.PC3(ADC3)
- new net A4-SDA: J2.14, U1.PC4(ADC4/SDA)
- new net A5-SCL: J2.13, U1.PC5(ADC5/SCL)
- new net ADC6: J2.12, U1.ADC6
- net 13: now also J2.5
- net 6V: now also J4.10, J4.11, J4.12, J4.13, J4.14, J4.15, J4.16, J4.17, J4.18, J4.5, J4.6, J4.7, J4.8, J4.9; no longer JP3.10, JP3.11, JP3.12, JP3.9
- net A0: now also J2.18
- net A1: now also J2.17
- net A2: now also J2.16
- net GND: now also J1.1, J1.10, J1.11, J1.12, J1.13, J1.14, J1.15, J1.16, J1.17, J1.18, J1.2, J1.3, J1.4, J1.5, J1.6, J1.7, J1.8, J1.9; no longer JP2.1, JP2.10, JP2.11, JP2.12, JP2.2, JP2.3, JP2.4, JP2.5, JP2.6, JP2.7, JP2.8, JP2.9
- net PIN_PWR: now also J4.1, J4.2, J4.3, J4.4; no longer JP3.1, JP3.2, JP3.3, JP3.4, JP3.5, JP3.6, JP3.7, JP3.8

Commit message: Routing BoB board
Parts:
- removed C4: 0.1uF, resistor:C-USC0805K
- removed Q9: MOSFET-NCHANNELAO3404A, SparkFun-DiscreteSemi:MOSFET-NCHANNELAO3404A
- removed R19, R21: 10k, resistor:R-US_R0805W
- added R3: 20k, resistor:R-US_R0805W
- added R4: 10k, resistor:R-US_R0805W
- R11, R12, R13: value 100k -> 470
Connections:
- net N$1 renamed AREF
- removed net N$12: Q1.S, R22.1, U$1.2-TX
- removed net N$15: Q9.S, R21.1, U$1.4-RX
- removed net N$9: LED1.RED-C, R13.2
- new net CONN_LED: LED1.RED-A, U$1.15-CONN_LED
- new net N$1: LED1.RED-C, R13.1
- new net U1_RX: Q1.D, R20.1, U1.PD1(TXD)
- new net U1_TX: R4.2, U1.PD0(RXD)
- new net U2-RESET: R1.2, U$1.11-RESET
- net 13: no longer LED1.RED-A
- net 3.35V: now also LED1.BLU-A, LED1.GRN-A; no longer Q9.G, R21.2
- net 3~: now also J2.18; no longer J2.11
- net 4: now also J2.17; no longer J2.10
- net A0: now also J2.12; no longer J2.18
- net A1: now also J2.10; no longer J2.17, LED1.GRN-A, U1.PC1(ADC1)
- net A2: no longer LED1.BLU-A, U1.PC2(ADC2)
- net ADC6: now also J2.11; no longer J2.12
- net GND: now also R13.2, R3.2; no longer C4.2, R11.1, R12.1, R13.1
- net RESET: no longer R1.2, U$1.11-RESET
- net U2_RX: now also R12.1, R3.1, R4.1, U$1.4-RX; no longer Q1.D, R20.1, U1.PD1(TXD)
- net U2_TX: now also Q1.S, R11.1, R22.1, U$1.2-TX; no longer Q9.D, R19.1, U1.PD0(RXD)
- net VCC: no longer C4.1, R19.2
Other:
- moved on the sheet: R1, R11, R12, R13, R20

Commit message: Finished routing BoB Board
Parts:
- removed C5: 0.1uF, resistor:C-USC0805K
Connections:
- removed net DTR: C5.1
- net A1: now also U1.PC1(ADC1)
- net A2: now also U1.PC2(ADC2)
- net A3: now also J2.13; no longer J2.15
- net A5-SCL: now also J2.15; no longer J2.13
- net RESET: no longer C5.2
Changed lines of the file:
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@@
 <part name="GND13" library="SparkFun-Aesthetics" deviceset="GND" device=""/>
 <part name="S1" library="SparkFun-Retired" deviceset="TAC_SWITCH" device="SMD" value="TAC_SWITCHSMD"/>
-<part name="C5" library="resistor" deviceset="C-US" device="C0805K" value="0.1uF"/>
 <part name="R14" library="resistor" deviceset="R-US_" device="R0805W" value="10k"/>
 <part name="SUPPLY4" library="SparkFun-Aesthetics" deviceset="VCC" device=""/>
@@
 <pinref part="J4" gate="G$1" pin="3"/>
 <junction x="20.32" y="2.54"/>
+<junction x="20.32" y="5.08"/>
 </segment>
 </net>
@@
 <net name="A3" class="0">
 <segment>
-<pinref part="J2" gate="G$1" pin="15"/>
-<wire x1="10.16" y1="-22.86" x2="2.54" y2="-22.86" width="0.1524" layer="91"/>
+<pinref part="J2" gate="G$1" pin="13"/>
+<wire x1="10.16" y1="-27.94" x2="2.54" y2="-27.94" width="0.1524" layer="91"/>
 <label x="2.54" y="-22.86" size="1.778" layer="95"/>
 </segment>
@@
 <net name="A5-SCL" class="0">
 <segment>
-<pinref part="J2" gate="G$1" pin="13"/>
-<wire x1="10.16" y1="-27.94" x2="2.54" y2="-27.94" width="0.1524" layer="91"/>
+<pinref part="J2" gate="G$1" pin="15"/>
+<wire x1="10.16" y1="-22.86" x2="2.54" y2="-22.86" width="0.1524" layer="91"/>
 <label x="2.54" y="-27.94" size="1.778" layer="95"/>
 </segment>
@@
 <instance part="GND13" gate="1" x="147.32" y="15.24" rot="MR0"/>
 <instance part="S1" gate="S" x="157.48" y="73.66"/>
-<instance part="C5" gate="G$1" x="162.56" y="83.82"/>
 <instance part="R14" gate="G$1" x="177.8" y="71.12"/>
 <instance part="SUPPLY4" gate="G$1" x="185.42" y="71.12" rot="R270"/>
@@
 </segment>
 </net>
-<net name="DTR" class="0">
-<segment>
-<pinref part="C5" gate="G$1" pin="1"/>
-<wire x1="162.56" y1="86.36" x2="162.56" y2="91.44" width="0.1524" layer="91"/>
-<label x="160.02" y="91.44" size="1.778" layer="95"/>
-</segment>
-</net>
 <net name="13" class="0">
 <segment>
@@
 <wire x1="109.22" y1="177.8" x2="109.22" y2="175.26" width="0.1524" layer="91"/>
 <label x="119.38" y="177.8" size="1.778" layer="95" xref="yes"/>
+<junction x="109.22" y="177.8"/>
 </segment>
 <segment>
@@
 <wire x1="198.12" y1="109.22" x2="198.12" y2="119.38" width="0.1524" layer="91"/>
 <label x="198.12" y="119.38" size="1.778" layer="95" rot="R90" xref="yes"/>
+<junction x="195.58" y="109.22"/>
 </segment>
 </net>
@@
 <net name="RESET" class="0">
 <segment>
-<pinref part="C5" gate="G$1" pin="2"/>
 <pinref part="S1" gate="S" pin="3"/>
-<wire x1="162.56" y1="73.66" x2="162.56" y2="78.74" width="0.1524" layer="91"/>
-<junction x="162.56" y="73.66"/>
 <pinref part="R14" gate="G$1" pin="1"/>
 <pinref part="S1" gate="S" pin="4"/>
@@
 </segment>
 </net>
+<net name="A1" class="0">
+<segment>
+<pinref part="U1" gate="U$1" pin="PC1(ADC1)"/>
+<wire x1="213.36" y1="50.8" x2="220.98" y2="50.8" width="0.1524" layer="91"/>
+<label x="213.36" y="50.8" size="1.778" layer="95"/>
+</segment>
+</net>
+<net name="A2" class="0">
+<segment>
+<pinref part="U1" gate="U$1" pin="PC2(ADC2)"/>
+<wire x1="213.36" y1="48.26" x2="220.98" y2="48.26" width="0.1524" layer="91"/>
+<label x="213.36" y="48.26" size="1.778" layer="95"/>
+</segment>
+</net>
