File: UART Splitter/UART_Splitter.sch (EAGLE design)
At the start: 6 parts, among them IC1 ATTINY10, U1 74HC4052

Commit message: UART Splitter
Parts:
- added C1, C2: 22pf, resistor:C-USC0805K
- added C3, C4, C5: 1uF, resistor:C-USC0805K
- added LED1, LED2, LED3, LED4, LED5, LED6, LED7, LED8: (no value), led:LEDSML0603
- added Q1: 12mhz, crystal:CRYSTALHC49UP
- added R1, R2, R3: 10k, resistor:R-US_R0805W
- added R10, R11, R4, R5, R6, R7, R8, R9: (no value), resistor:R-US_R0805W
Connections:
- net N$8 renamed TX
- net N$9 renamed RX
- new net N$10: C2.1, Q1.1, U$1.XI
- new net N$11: C1.1, Q1.2, U$1.XO
- new net N$12: IC1.PB2, R3.2
- new net N$14: LED8.A, R4.1
- new net N$15: LED7.A, R5.1
- new net N$16: LED6.A, R6.1
- new net N$17: LED5.A, R7.1
- new net N$18: LED4.A, R8.1
- new net N$19: LED3.A, R9.1
- new net N$20: LED2.A, R10.1
- new net N$21: LED1.A, R11.1
- new net N$5: R2.1, U1.A
- new net N$6: R1.1, U1.B
- new net N$7: U1.INH
- new net N$8: IC1.PB0, R1.2
- new net N$9: IC1.PB1, R2.2
- new net RX0: JP3.1, LED1.C, U1.Y0
- new net RX1: JP3.5, U1.Y1
- new net RX2: JP2.1, U1.Y2
- new net RX3: JP2.5, U1.Y3
- new net TX0: JP3.2, U1.X0
- new net TX1: JP3.6, U1.X1
- new net TX2: JP2.2, U1.X2
- new net TX3: JP2.6, U1.X3
- new net VCC: JP2.4, JP2.8, JP3.4, JP3.8, R10.2, R11.2, R4.2, R5.2, R6.2, R7.2, R8.2, R9.2
- net GND: now also C1.2, C2.2, C3.2, C4.2, C5.2, JP2.3, JP2.7, JP3.3, JP3.7
- net N$2: now also C3.1, C4.1, C5.1
Other:
- moved on the sheet: IC1, JP2, JP3, U1

Commit message: UART Splitter
Parts:
- added R12: 10k, resistor:R-US_R0402
- added S1: (no value), SparkFun-Electromechanical:TAC_SWITCHSMD
- C1, C2, C3, C4, C5: device resistor:C-USC0805K -> resistor:C-USC0402K
- R1, R10, R11, R2, R3, R4, R5, R6, R7, R8, R9: device resistor:R-US_R0805W -> resistor:R-US_R0402
Connections:
- new net N$13: R12.1, U1.INH
- net GND: now also S1.3, S1.4
- net N$2: now also R1.2
- net N$6: no longer R1.1
- net N$7: now also IC1.PB1, R1.1, S1.1, S1.2; no longer U1.INH
- net N$8: now also IC1./RST, R12.2; no longer IC1.PB0, R1.2
- net N$9: now also IC1.PB0; no longer IC1.PB1
Other:
- moved on the sheet: JP2, JP3, R1

Commit message: UART Splitter
Connections:
- net N$14 renamed LED_TX3
- net N$15 renamed LED_RX3
- net N$16 renamed LED_TX2
- net N$17 renamed LED_RX2
- net N$18 renamed LED_TX1
- net N$19 renamed LED_RX1
- net N$20 renamed LED_TX0
- net N$21 renamed LED_RX0
- removed net N$1: U$1.GND, U$2.GND
- removed net N$2: C3.1, C4.1, C5.1, IC1.VCC, R1.2, U$1.VCC, U$2.VBUS, U1.VCC
- net GND: now also U$1.GND, U$2.GND
- net N$6: now also R3.1
- net RX1: now also LED3.C
- net RX2: now also LED5.C
- net RX3: now also LED7.C
- net TX0: now also LED2.C
- net TX1: now also LED4.C
- net TX2: now also LED6.C
- net TX3: now also LED8.C
- net VCC: now also C3.1, C4.1, C5.1, IC1.VCC, R1.2, U$1.VCC, U$2.VBUS, U1.VCC
Other:
- moved on the sheet: R2

Commit message: UART
Parts:
- LED1, LED3, LED5, LED7: value (none) -> GREEN
- LED2, LED4, LED6, LED8: value (none) -> BLUE
- R10, R11, R4, R5, R6, R7, R8, R9: value (none) -> 330
Changed lines of the file:
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@@
 <part name="R2" library="resistor" deviceset="R-US_" device="R0402" value="10k"/>
 <part name="R3" library="resistor" deviceset="R-US_" device="R0402" value="10k"/>
-<part name="R4" library="resistor" deviceset="R-US_" device="R0402"/>
-<part name="R5" library="resistor" deviceset="R-US_" device="R0402"/>
-<part name="R6" library="resistor" deviceset="R-US_" device="R0402"/>
-<part name="R7" library="resistor" deviceset="R-US_" device="R0402"/>
-<part name="R8" library="resistor" deviceset="R-US_" device="R0402"/>
-<part name="R9" library="resistor" deviceset="R-US_" device="R0402"/>
-<part name="R10" library="resistor" deviceset="R-US_" device="R0402"/>
-<part name="R11" library="resistor" deviceset="R-US_" device="R0402"/>
-<part name="LED1" library="led" deviceset="LED" device="SML0603"/>
-<part name="LED2" library="led" deviceset="LED" device="SML0603"/>
-<part name="LED3" library="led" deviceset="LED" device="SML0603"/>
-<part name="LED4" library="led" deviceset="LED" device="SML0603"/>
-<part name="LED5" library="led" deviceset="LED" device="SML0603"/>
-<part name="LED6" library="led" deviceset="LED" device="SML0603"/>
-<part name="LED7" library="led" deviceset="LED" device="SML0603"/>
-<part name="LED8" library="led" deviceset="LED" device="SML0603"/>
+<part name="R4" library="resistor" deviceset="R-US_" device="R0402" value="330"/>
+<part name="R5" library="resistor" deviceset="R-US_" device="R0402" value="330"/>
+<part name="R6" library="resistor" deviceset="R-US_" device="R0402" value="330"/>
+<part name="R7" library="resistor" deviceset="R-US_" device="R0402" value="330"/>
+<part name="R8" library="resistor" deviceset="R-US_" device="R0402" value="330"/>
+<part name="R9" library="resistor" deviceset="R-US_" device="R0402" value="330"/>
+<part name="R10" library="resistor" deviceset="R-US_" device="R0402" value="330"/>
+<part name="R11" library="resistor" deviceset="R-US_" device="R0402" value="330"/>
+<part name="LED1" library="led" deviceset="LED" device="SML0603" value="GREEN"/>
+<part name="LED2" library="led" deviceset="LED" device="SML0603" value="BLUE"/>
+<part name="LED3" library="led" deviceset="LED" device="SML0603" value="GREEN"/>
+<part name="LED4" library="led" deviceset="LED" device="SML0603" value="BLUE"/>
+<part name="LED5" library="led" deviceset="LED" device="SML0603" value="GREEN"/>
+<part name="LED6" library="led" deviceset="LED" device="SML0603" value="BLUE"/>
+<part name="LED7" library="led" deviceset="LED" device="SML0603" value="GREEN"/>
+<part name="LED8" library="led" deviceset="LED" device="SML0603" value="BLUE"/>
 <part name="S1" library="SparkFun-Electromechanical" deviceset="TAC_SWITCH" device="SMD"/>
 <part name="R1" library="resistor" deviceset="R-US_" device="R0402" value="10k"/>
@@
 <junction x="-33.02" y="119.38"/>
 <pinref part="GND1" gate="1" pin="GND"/>
+<junction x="-30.48" y="139.7"/>
+<junction x="-33.02" y="139.7"/>
 </segment>
 <segment>
@@
 <wire x1="114.3" y1="109.22" x2="114.3" y2="104.14" width="0.1524" layer="91"/>
 <pinref part="GND8" gate="1" pin="GND"/>
+<junction x="114.3" y="109.22"/>
+<junction x="114.3" y="111.76"/>
 </segment>
 <segment>
@@
 <wire x1="71.12" y1="111.76" x2="71.12" y2="109.22" width="0.1524" layer="91"/>
 <junction x="71.12" y="109.22"/>
-</segment>
-</net>
+<junction x="104.14" y="109.22"/>
+<junction x="104.14" y="111.76"/>
+</segment>
+</net>
