File: micro-stepper-driver/micro-stepper-driver-v1.brd (EAGLE design)
At the start: 11.1 x 12.7 mm, 3 parts

Commit message: Micro driver
Parts:
- removed J1, J2: (no value), SparkFun-Connectors:1X06
- added C1, C2: 10uF, SparkFun-Capacitors:EIA3216
- added C3, C4: 1uF, resistor:C0805K
- added U$2: EDGE_MOUNT_HEADER_X10, Ladvien_Eagle_Parts:EDGE_MOUNT_HEAD_X10
- added U$3: EDGE_MOUNT_HEAD_X8, Ladvien_Eagle_Parts:EDGE_MOUNT_HEAD_X8
- added U$4: DRV8835, Ladvien_Eagle_Parts:DRV8835
- moved U$1 12.9 mm to (12.2, 17.1), turned to 180 degrees
Connections:
- removed net N$1: J1.1, U$1.6, U$1.PAD
- removed net N$10: J2.4, U$1.9
- removed net N$11: J2.5, U$1.8
- removed net N$12: J2.6, U$1.7
- removed net N$2: J1.2, U$1.5
- removed net N$3: J1.3, U$1.4
- removed net N$4: J1.4, U$1.3
- removed net N$5: J1.5, U$1.2
- removed net N$6: J1.6, U$1.1
- removed net N$7: J2.1, U$1.12
- removed net N$8: J2.2, U$1.11
- removed net N$9: J2.3, U$1.10
- new net 1AIN1: U$2.8, U$4.10
- new net 1AIN2: U$2.7, U$4.9
- new net 1AOUT1: U$3.1, U$4.2
- new net 1AOUT2: U$3.2, U$4.3
- new net 1BIN1: U$2.6, U$4.8
- new net 1BIN2: U$2.5, U$4.7
- new net 1BOUT1: U$3.3, U$4.4
- new net 1BOUT2: U$3.4, U$4.5
- new net 2AIN1: U$1.10, U$2.4
- new net 2AIN2: U$1.9, U$2.3
- new net 2AOUT1: U$1.2, U$3.5
- new net 2AOUT2: U$1.3, U$3.6
- new net 2BIN1: U$1.8, U$2.2
- new net 2BIN2: U$1.7, U$2.1
- new net 2BOUT1: U$1.4, U$3.7
- new net 2BOUT2: U$1.5, U$3.8
- new net GND: C1.-, C2.-, C3.2, C4.2, U$1.11, U$1.6, U$1.PAD, U$2.9, U$4.11, U$4.6, U$4.PAD
- new net VCC/VM: C1.+, C2.+, C3.1, C4.1, U$1.1, U$1.12, U$2.10, U$4.1, U$4.12
Routing:
- net VCC/VM: track 0.00 -> 35.1 mm, vias 0 -> 2
- net 2BIN2: track 0.00 -> 13.5 mm
- net 1BIN2: track 0.00 -> 13.0 mm
- net 2BIN1: track 0.00 -> 12.7 mm
- net 1BIN1: track 0.00 -> 12.2 mm
- net 2AIN2: track 0.00 -> 11.8 mm
- net 1AIN1: track 0.00 -> 11.8 mm
- net 1AIN2: track 0.00 -> 11.4 mm
- net 2AIN1: track 0.00 -> 11.3 mm
- net 2BOUT2: track 0.00 -> 8.95 mm
- net 1AOUT1: track 0.00 -> 8.75 mm
- net 1BOUT2: track 0.00 -> 7.88 mm
- net 2AOUT1: track 0.00 -> 7.83 mm
- net 2BOUT1: track 0.00 -> 7.51 mm
- net 1AOUT2: track 0.00 -> 7.46 mm
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- added copper zone on layer 1, net GND
- added copper zone on layer 16, net GND
Other:
- board size 11.1 x 12.7 mm -> 25.8 x 25.4 mm

Commit message: MicroStepper
Parts:
- removed C3, C4: 1uF, resistor:C0805K
- added C6: 1000uF, resistor:153CLV-0810
- added D1: 20V-1A, Seeed-Diode:SOD-123
- added LED1: GREEN, led:SML0603
- added R1: 330, resistor:R0402
- C1, C2: value 10uF -> (none); device SparkFun-Capacitors:EIA3216 -> resistor:C0402K
- moved C1 7.74 mm to (16.3, 9.40), turned to 270 degrees
- moved C2 5.85 mm to (16.0, 16.3), turned to 270 degrees
- moved U$4 5.14 mm to (14.0, 13.0)
- moved U$1 3.30 mm to (10.9, 20.2)
Connections:
- new net N$2: LED1.C, R1.2
- new net VIN: D1.+, U$2.10
- net GND: now also C1.2, C2.2, C6.-, R1.1; no longer C1.-, C2.-, C3.2, C4.2
- net VCC/VM: now also C1.1, C2.1, C6.+, D1.-, LED1.A; no longer C1.+, C2.+, C3.1, C4.1, U$2.10
Routing:
- net N$1: track 0.00 -> 8.64 mm
- net VIN: track 0.00 -> 7.54 mm
- net 1AIN1: track 11.8 -> 17.2 mm
- net VCC/VM: track 35.1 -> 30.8 mm
- net 1AOUT1: track 8.75 -> 12.8 mm
- net 1AIN2: track 11.4 -> 15.4 mm
- net 2AOUT1: track 7.83 -> 11.8 mm
- net 1AOUT2: track 7.46 -> 10.4 mm
- net 2AOUT2: track 6.98 -> 9.52 mm
- net 2BIN1: track 12.7 -> 10.1 mm
- net 2BIN2: track 13.5 -> 11.2 mm
- net 1BOUT2: track 7.88 -> 5.99 mm
- net 2AIN2: track 11.8 -> 10.1 mm
- net 1BIN1: track 12.2 -> 13.9 mm
- net N$2: track 0.00 -> 1.59 mm
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Other:
- board text added: "Thomas Brittain (c) aka, Ladvien MicroDriver v01"
